File: hardware/wasp_node_board/eth.kicad_sch (KiCad schematic)
At the start: 51 parts, among them J2 RJ45_Hanrun_HR911105A_Horizon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, J4 RJ45_Hanrun_HR911105A_Horizon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, J5 RJ45_Hanrun_HR911105A_Horizon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, U5 KSZ8794CNXCC, Y1 TSX-3225 25.00M-N0YYYYG30RGB

Commit message: V1 layout done
Changed lines of the file:
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@@
 					(size 1.27 1.27)
 				)
+				(hide yes)
 			)
 		)
@@
 					(size 1.27 1.27)
 				)
+				(hide yes)
 			)
 		)
@@
 					(size 1.27 1.27)
 				)
+				(hide yes)
 			)
 		)
@@
 					(size 1.27 1.27)
 				)
+				(hide yes)
 			)
 		)
@@
 					(size 1.27 1.27)
 				)
+				(hide yes)
 			)
 		)
@@
 					(size 1.27 1.27)
 				)
+				(hide yes)
 			)
 		)
@@
 					(size 1.27 1.27)
 				)
+				(hide yes)
 			)
 		)
@@
 					(size 1.27 1.27)
 				)
+				(hide yes)
 			)
 		)
@@
 					(size 1.27 1.27)
 				)
+				(hide yes)
 			)
 		)
@@
 					(size 1.27 1.27)
 				)
+				(hide yes)
 			)
 		)
@@
 					(size 1.27 1.27)
 				)
+				(hide yes)
 			)
 		)

Commit message: Order of the V1 board done
Parts:
- Y1: value TSX-3225 25.00M-N0YYYYG30RGB -> TSX-3225 25.0000MF20P-C0
Changed lines of the file:
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@@
 			)
 		)
-		(property "Value" "TSX-3225 25.00M-N0YYYYG30RGB"
+		(property "Value" "TSX-3225 25.0000MF20P-C0"
 			(at 31.75 154.94 0)
 			(effects
